Commit message: Faz 2: ros2_control + diff_drive + clock bridge, rover moves with real odometry

File: src/rover_description/urdf/rover.urdf.xacro (robot description, xacro)
@@ -91,3 +91,47 @@
   <xacro:wheel prefix="rear_left"   x_offset="${-wheel_offset_x}" y_offset="${ wheel_offset_y}"/>
   <xacro:wheel prefix="rear_right"  x_offset="${-wheel_offset_x}" y_offset="${-wheel_offset_y}"/>
+<!-- ===== ros2_control HARDWARE TANIMI ===== -->
+  <ros2_control name="GazeboSystem" type="system">
+    <hardware>
+      <plugin>gz_ros2_control/GazeboSimSystem</plugin>
+    </hardware>
+    <joint name="front_left_wheel_joint">
+      <command_interface name="velocity">
+        <param name="min">-10.0</param>
+        <param name="max"> 10.0</param>
+      </command_interface>
+      <state_interface name="position"/>
+      <state_interface name="velocity"/>
+    </joint>
+    <joint name="front_right_wheel_joint">
+      <command_interface name="velocity">
+        <param name="min">-10.0</param>
+        <param name="max"> 10.0</param>
+      </command_interface>
+      <state_interface name="position"/>
+      <state_interface name="velocity"/>
+    </joint>
+    <joint name="rear_left_wheel_joint">
+      <command_interface name="velocity">
+        <param name="min">-10.0</param>
+        <param name="max"> 10.0</param>
+      </command_interface>
+      <state_interface name="position"/>
+      <state_interface name="velocity"/>
+    </joint>
+    <joint name="rear_right_wheel_joint">
+      <command_interface name="velocity">
+        <param name="min">-10.0</param>
+        <param name="max"> 10.0</param>
+      </command_interface>
+      <state_interface name="position"/>
+      <state_interface name="velocity"/>
+    </joint>
+  </ros2_control>
+  <!-- ===== GAZEBO PLUGIN (controller manager Gazebo içinde çalışsın) ===== -->
+  <gazebo>
+    <plugin filename="gz_ros2_control-system" name="gz_ros2_control::GazeboSimROS2ControlPlugin">
+      <parameters>$(find rover_control)/config/controllers.yaml</parameters>
+    </plugin>
+  </gazebo>
 </robot>

Commit message: Faz 3: IMU + camera + GPS sensors integrated and verified

File: src/rover_description/urdf/rover.urdf.xacro (robot description, xacro)
@@ -135,3 +135,136 @@
     </plugin>
   </gazebo>
+  <!-- ===== IMU LINK ===== -->
+  <link name="imu_link">
+    <inertial>
+      <mass value="0.001"/>
+      <inertia ixx="1e-9" ixy="0" ixz="0" iyy="1e-9" iyz="0" izz="1e-9"/>
+    </inertial>
+    <visual>
+      <geometry>
+        <box size="0.02 0.02 0.005"/>
+      </geometry>
+      <material name="imu_red"><color rgba="0.8 0.1 0.1 1.0"/></material>
+    </visual>
+  </link>
+  <joint name="imu_joint" type="fixed">
+    <parent link="base_link"/>
+    <child link="imu_link"/>
+    <origin xyz="0 0 ${chassis_height/2 + 0.005}" rpy="0 0 0"/>
+  </joint>
+  <!-- ===== GAZEBO IMU SENSÖRÜ ===== -->
+  <gazebo reference="imu_link">
+    <sensor name="imu_sensor" type="imu">
+      <always_on>true</always_on>
+      <update_rate>100</update_rate>
+      <topic>imu</topic>
+      <gz_frame_id>imu_link</gz_frame_id>
+      <imu>
+        <angular_velocity>
+          <x><noise type="gaussian"><mean>0.0</mean><stddev>2e-4</stddev></noise></x>
+          <y><noise type="gaussian"><mean>0.0</mean><stddev>2e-4</stddev></noise></y>
+          <z><noise type="gaussian"><mean>0.0</mean><stddev>2e-4</stddev></noise></z>
+        </angular_velocity>
+        <linear_acceleration>
+          <x><noise type="gaussian"><mean>0.0</mean><stddev>1.7e-2</stddev></noise></x>
+          <y><noise type="gaussian"><mean>0.0</mean><stddev>1.7e-2</stddev></noise></y>
+          <z><noise type="gaussian"><mean>0.0</mean><stddev>1.7e-2</stddev></noise></z>
+        </linear_acceleration>
+      </imu>
+    </sensor>
+  </gazebo>
+  <!-- ===== KAMERA LINK (gövde frame'i) ===== -->
+  <link name="camera_link">
+    <inertial>
+      <mass value="0.001"/>
+      <inertia ixx="1e-9" ixy="0" ixz="0" iyy="1e-9" iyz="0" izz="1e-9"/>
+    </inertial>
+    <visual>
+      <geometry>
+        <box size="0.025 0.03 0.02"/>
+      </geometry>
+      <material name="camera_grey"><color rgba="0.2 0.2 0.2 1.0"/></material>
+    </visual>
+  </link>
+  <joint name="camera_joint" type="fixed">
+    <parent link="base_link"/>
+    <child link="camera_link"/>
+    <!-- Şasinin önüne, ortaya, hafif yukarı -->
+    <origin xyz="${chassis_length/2 - 0.015} 0 ${chassis_height/2 + 0.015}" rpy="0 0 0"/>
+  </joint>
+  <!-- ===== KAMERA OPTİK FRAME'İ ===== -->
+  <!-- ROS gövde konvansiyonu (X ileri, Y sol, Z yukarı) ile
+       optik konvansiyon (X sağ, Y aşağı, Z ileri) arasındaki dönüşüm -->
+  <link name="camera_link_optical"/>
+  <joint name="camera_optical_joint" type="fixed">
+    <parent link="camera_link"/>
+    <child link="camera_link_optical"/>
+    <origin xyz="0 0 0" rpy="${-pi/2} 0 ${-pi/2}"/>
+  </joint>
+  <!-- ===== GAZEBO KAMERA SENSÖRÜ ===== -->
+  <gazebo reference="camera_link">
+    <sensor name="rgb_camera" type="camera">
+      <always_on>true</always_on>
+      <update_rate>30</update_rate>
+      <visualize>true</visualize>
+      <topic>camera/image_raw</topic>
+      <gz_frame_id>camera_link_optical</gz_frame_id>
+      <camera>
+        <horizontal_fov>1.396</horizontal_fov>  <!-- ~80 derece, geniş FPV açısı -->
+        <image>
+          <width>640</width>
+          <height>480</height>
+          <format>R8G8B8</format>
+        </image>
+        <clip>
+          <near>0.05</near>
+          <far>100</far>
+        </clip>
+      </camera>
+    </sensor>
+  </gazebo>
+  <!-- ===== GPS LINK ===== -->
+  <link name="gps_link">
+    <inertial>
+      <mass value="0.001"/>
+      <inertia ixx="1e-9" ixy="0" ixz="0" iyy="1e-9" iyz="0" izz="1e-9"/>
+    </inertial>
+    <visual>
+      <geometry>
+        <cylinder radius="0.01" length="0.005"/>
+      </geometry>
+      <material name="gps_yellow"><color rgba="0.9 0.8 0.1 1.0"/></material>
+    </visual>
+  </link>
+  <joint name="gps_joint" type="fixed">
+    <parent link="base_link"/>
+    <child link="gps_link"/>
+    <!-- Şasinin üzerinde, arka kısma yakın -->
+    <origin xyz="${-chassis_length/2 + 0.04} 0 ${chassis_height/2 + 0.01}" rpy="0 0 0"/>
+  </joint>
+  <!-- ===== GAZEBO NAVSAT SENSÖRÜ ===== -->
+  <gazebo reference="gps_link">
+    <sensor name="navsat_sensor" type="navsat">
+      <always_on>true</always_on>
+      <update_rate>10</update_rate>
+      <topic>gps</topic>
+      <gz_frame_id>gps_link</gz_frame_id>
+      <navsat>
+        <position_sensing>
+          <horizontal>
+            <noise type="gaussian">
+              <mean>0.0</mean>
+              <stddev>0.00001</stddev>     <!-- ≈1m yatay noise (1e-5 derece) -->
+            </noise>
+          </horizontal>
+          <vertical>
+            <noise type="gaussian">
+              <mean>0.0</mean>
+              <stddev>1.5</stddev>          <!-- 1.5m dikey, gerçek GPS tipik -->
+            </noise>
+          </vertical>
+        </position_sensing>
+      </navsat>
+    </sensor>
+  </gazebo>
 </robot>

Commit message: Faz 5 complete: box-based terrain, dartsim with anisotropic wheel friction (mu1=0.7, mu2=0.25), IMU pitch matches ramp angles ±0.1°, Z accel matches gravity projection

File: src/rover_description/urdf/rover.urdf.xacro (robot description, xacro)
@@ -1,28 +1,30 @@
 <?xml version="1.0"?>
-<robot name="rover" xmlns:xacro="http://www.ros.org/wiki/xacro">
+<robot name="rover"
+  xmlns:xacro="http://www.ros.org/wiki/xacro">
   <!-- ===== KİTE GÖRE PARAMETRELER (ANIM 4WD) ===== -->
   <!-- Şasi: 25.5 x 15 cm akrilik, çift kat + motorlar arası -->
   <xacro:property name="chassis_length" value="0.255"/>
-  <xacro:property name="chassis_width"  value="0.15"/>
+  <xacro:property name="chassis_width" value="0.15"/>
   <xacro:property name="chassis_height" value="0.06"/>
-  <xacro:property name="chassis_mass"   value="0.8"/>
+  <xacro:property name="chassis_mass" value="0.8"/>
   <!-- Teker: 6.5 cm çap, 2.7 cm genişlik -->
   <xacro:property name="wheel_radius" value="0.0325"/>
-  <xacro:property name="wheel_width"  value="0.027"/>
-  <xacro:property name="wheel_mass"   value="0.03"/>
+  <xacro:property name="wheel_width" value="0.027"/>
+  <xacro:property name="wheel_mass" value="0.03"/>
   <!-- Teker yerleşimi (şasi merkezinden) -->
   <xacro:property name="wheel_offset_x" value="0.09"/>
   <xacro:property name="wheel_offset_y" value="0.095"/>
   <!-- ===== MATERYALLER ===== -->
-  <material name="acrylic_blue"><color rgba="0.2 0.4 0.8 0.85"/></material>
-  <material name="tire_black"><color rgba="0.1 0.1 0.1 1.0"/></material>
+  <material name="acrylic_blue">
+    <color rgba="0.2 0.4 0.8 0.85"/>
+  </material>
+  <material name="tire_black">
+    <color rgba="0.1 0.1 0.1 1.0"/>
+  </material>
   <!-- ===== INERTIA MACRO'LARI ===== -->
   <xacro:macro name="box_inertia" params="m x y z">
     <inertial>
       <mass value="${m}"/>
-      <inertia
-        ixx="${(1/12) * m * (y*y + z*z)}" ixy="0" ixz="0"
-        iyy="${(1/12) * m * (x*x + z*z)}" iyz="0"
-        izz="${(1/12) * m * (x*x + y*y)}"/>
+      <inertia ixx="${(1/12) * m * (y*y + z*z)}" ixy="0" ixz="0" iyy="${(1/12) * m * (x*x + z*z)}" iyz="0" izz="${(1/12) * m * (x*x + y*y)}"/>
     </inertial>
   </xacro:macro>
@@ -30,8 +32,5 @@
     <inertial>
       <mass value="${m}"/>
-      <inertia
-        ixx="${(1/12) * m * (3*r*r + h*h)}" ixy="0" ixz="0"
-        iyy="${(1/2) * m * r*r}"            iyz="0"
-        izz="${(1/12) * m * (3*r*r + h*h)}"/>
+      <inertia ixx="${(1/12) * m * (3*r*r + h*h)}" ixy="0" ixz="0" iyy="${(1/2) * m * r*r}" iyz="0" izz="${(1/12) * m * (3*r*r + h*h)}"/>
     </inertial>
   </xacro:macro>
@@ -50,12 +49,9 @@
       </geometry>
     </collision>
-    <xacro:box_inertia m="${chassis_mass}"
-                       x="${chassis_length}"
-                       y="${chassis_width}"
-                       z="${chassis_height}"/>
+    <xacro:box_inertia m="${chassis_mass}" x="${chassis_length}" y="${chassis_width}" z="${chassis_height}"/>
   </link>
   <joint name="base_footprint_to_base_link" type="fixed">
     <parent link="base_footprint"/>
-    <child  link="base_link"/>
+    <child link="base_link"/>
     <origin xyz="0 0 ${wheel_radius + chassis_height/2}" rpy="0 0 0"/>
   </joint>
@@ -76,20 +72,18 @@
         </geometry>
       </collision>
-      <xacro:cylinder_inertia m="${wheel_mass}"
-                              r="${wheel_radius}"
-                              h="${wheel_width}"/>
+      <xacro:cylinder_inertia m="${wheel_mass}" r="${wheel_radius}" h="${wheel_width}"/>
     </link>
     <joint name="${prefix}_wheel_joint" type="continuous">
       <parent link="base_link"/>
-      <child  link="${prefix}_wheel"/>
+      <child link="${prefix}_wheel"/>
       <origin xyz="${x_offset} ${y_offset} ${-chassis_height/2}" rpy="0 0 0"/>
       <axis xyz="0 1 0"/>
     </joint>
   </xacro:macro>
-  <xacro:wheel prefix="front_left"  x_offset="${ wheel_offset_x}" y_offset="${ wheel_offset_y}"/>
+  <xacro:wheel prefix="front_left" x_offset="${ wheel_offset_x}" y_offset="${ wheel_offset_y}"/>
   <xacro:wheel prefix="front_right" x_offset="${ wheel_offset_x}" y_offset="${-wheel_offset_y}"/>
-  <xacro:wheel prefix="rear_left"   x_offset="${-wheel_offset_x}" y_offset="${ wheel_offset_y}"/>
-  <xacro:wheel prefix="rear_right"  x_offset="${-wheel_offset_x}" y_offset="${-wheel_offset_y}"/>
-<!-- ===== ros2_control HARDWARE TANIMI ===== -->
+  <xacro:wheel prefix="rear_left" x_offset="${-wheel_offset_x}" y_offset="${ wheel_offset_y}"/>
+  <xacro:wheel prefix="rear_right" x_offset="${-wheel_offset_x}" y_offset="${-wheel_offset_y}"/>
+  <!-- ===== ros2_control HARDWARE TANIMI ===== -->
   <ros2_control name="GazeboSystem" type="system">
     <hardware>
@@ -145,5 +139,7 @@
         <box size="0.02 0.02 0.005"/>
       </geometry>
-      <material name="imu_red"><color rgba="0.8 0.1 0.1 1.0"/></material>
+      <material name="imu_red">
+        <color rgba="0.8 0.1 0.1 1.0"/>
+      </material>
     </visual>
   </link>
@@ -162,12 +158,42 @@
       <imu>
         <angular_velocity>
-          <x><noise type="gaussian"><mean>0.0</mean><stddev>2e-4</stddev></noise></x>
-          <y><noise type="gaussian"><mean>0.0</mean><stddev>2e-4</stddev></noise></y>
-          <z><noise type="gaussian"><mean>0.0</mean><stddev>2e-4</stddev></noise></z>
+          <x>
+            <noise type="gaussian">
+              <mean>0.0</mean>
+              <stddev>2e-4</stddev>
+            </noise>
+          </x>
+          <y>
+            <noise type="gaussian">
+              <mean>0.0</mean>
+              <stddev>2e-4</stddev>
+            </noise>
+          </y>
+          <z>
+            <noise type="gaussian">
+              <mean>0.0</mean>
+              <stddev>2e-4</stddev>
+            </noise>
+          </z>
         </angular_velocity>
         <linear_acceleration>
-          <x><noise type="gaussian"><mean>0.0</mean><stddev>1.7e-2</stddev></noise></x>
-          <y><noise type="gaussian"><mean>0.0</mean><stddev>1.7e-2</stddev></noise></y>
-          <z><noise type="gaussian"><mean>0.0</mean><stddev>1.7e-2</stddev></noise></z>
+          <x>
+            <noise type="gaussian">
+              <mean>0.0</mean>
+              <stddev>1.7e-2</stddev>
+            </noise>
+          </x>
+          <y>
+            <noise type="gaussian">
+              <mean>0.0</mean>
+              <stddev>1.7e-2</stddev>
+            </noise>
+          </y>
+          <z>
+            <noise type="gaussian">
+              <mean>0.0</mean>
+              <stddev>1.7e-2</stddev>
+            </noise>
+          </z>
         </linear_acceleration>
       </imu>
@@ -184,5 +210,7 @@
         <box size="0.025 0.03 0.02"/>
       </geometry>
-      <material name="camera_grey"><color rgba="0.2 0.2 0.2 1.0"/></material>
+      <material name="camera_grey">
+        <color rgba="0.2 0.2 0.2 1.0"/>
+      </material>
     </visual>
   </link>
@@ -211,5 +239,5 @@
       <gz_frame_id>camera_link_optical</gz_frame_id>
       <camera>
-        <horizontal_fov>1.396</horizontal_fov>  <!-- ~80 derece, geniş FPV açısı -->
+        <horizontal_fov>1.396</horizontal_fov>        <!-- ~80 derece, geniş FPV açısı -->
         <image>
           <width>640</width>
@@ -234,5 +262,7 @@
         <cylinder radius="0.01" length="0.005"/>
       </geometry>
-      <material name="gps_yellow"><color rgba="0.9 0.8 0.1 1.0"/></material>
+      <material name="gps_yellow">
+        <color rgba="0.9 0.8 0.1 1.0"/>
+      </material>
     </visual>
   </link>
@@ -255,5 +285,5 @@
             <noise type="gaussian">
               <mean>0.0</mean>
-              <stddev>0.00001</stddev>     <!-- ≈1m yatay noise (1e-5 derece) -->
+              <stddev>0.00001</stddev>              <!-- ≈1m yatay noise (1e-5 derece) -->
             </noise>
           </horizontal>
@@ -261,5 +291,5 @@
             <noise type="gaussian">
               <mean>0.0</mean>
-              <stddev>1.5</stddev>          <!-- 1.5m dikey, gerçek GPS tipik -->
+              <stddev>1.5</stddev>              <!-- 1.5m dikey, gerçek GPS tipik -->
             </noise>
           </vertical>
@@ -268,3 +298,18 @@
     </sensor>
   </gazebo>
+  <!-- ===== WHEEL FRICTION (skid-steer için ayarlı) ===== -->
+  <xacro:macro name="wheel_friction" params="prefix">
+    <gazebo reference="${prefix}_wheel">
+      <mu1>0.7</mu1>      <!-- yuvarlanma yönü: tutuş normal -->
+      <mu2>0.25</mu2>      <!-- yan yön: düşük, skid-steer kaymasına izin ver -->
+      <kp>1e7</kp>
+      <kd>1.0</kd>
+      <fdir1>1 0 0</fdir1>      <!-- birinci sürtünme ekseni: X (yuvarlanma) -->
+      <minDepth>0.001</minDepth>
+    </gazebo>
+  </xacro:macro>
+  <xacro:wheel_friction prefix="front_left"/>
+  <xacro:wheel_friction prefix="front_right"/>
+  <xacro:wheel_friction prefix="rear_left"/>
+  <xacro:wheel_friction prefix="rear_right"/>
 </robot>
